File: kicad/ledcube.kicad_sch (KiCad schematic)
At the start: 40 parts, among them P1 USB_C_Plug_USB2.0

Commit message: v1.2 LedCube pcb
Parts:
- added D10: LED, LED_SMD:LED_0805_2012Metric, symbol Device:LED
- added Q1, Q2, Q3: BC847, Package_TO_SOT_SMD:SOT-23, symbol Transistor_BJT:BC847
- added R28, R29, R30: 1000R, Resistor_SMD:R_0603_1608Metric, symbol Device:R
- added R31: 150R, Resistor_SMD:R_0603_1608Metric, symbol Device:R
- Blue1, Green1, Red1: footprint Potentiometer_THT:Potentiometer_Bourns_3266W_Vertical -> Potentiometer_SMD:Potentiometer_Bourns_3314G_Vertical
Connections:
- net at R12.2, R15.2, R18.2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: now also Q3.3 (C); no longer Blue1.1
- net at R1.2, R10.2, R13.2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: now also Q1.3 (C); no longer Green1.1
- net at D1.4 (AG), D1.5 (AR), D1.6 (AB)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: now also Blue1.1, Green1.1, Red1.1, R31.2
- net at R11.2, R14.2, R17.2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: now also Q2.3 (C); no longer Red1.1
- net at P1.A1 (GND), P1.A12 (GND), P1.B1 (GND)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: now also Blue1.3, Green1.3, Red1.3, D10.1 (K), Q1.2 (E), Q2.2 (E), Q3.2 (E); no longer Blue1.2, Green1.2, Red1.2
- new net: Green1.2, R28.1
- new net: Q1.1 (B), R28.2
- new net: R29.1, Red1.2
- new net: Q2.1 (B), R29.2
- new net: Blue1.2, R30.1
- new net: Q3.1 (B), R30.2
- new net: D10.2 (A), R31.1
Other:
- moved on the sheet: Blue1, Green1, Red1
