File: kicad/ledcube.kicad_pcb (KiCad board)
At the start: 2 copper layers, 45 x 45 mm, 49 parts, among them P1 USB_C_Plug_USB2.0, SW1 SW_SPDT_321, SW2 SW_SPDT_321, SW3 SW_SPDT_321

Commit message: Fixed bugs on PCB & 3d models
Routing:
- net Net-(D2-KG): track 0.00 -> 2.73 mm
Changed lines of the file:
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@@
+	)
+	(segment
+		(start 86.35 80.8)
+		(end 86.15 81)
+		(width 0.2)
+		(layer "F.Cu")
+		(net "Net-(D2-KG)")
+	)
+	(segment
+		(start 88.8 80.8)
+		(end 86.35 80.8)
+		(width 0.2)
+		(layer "F.Cu")
+		(net "Net-(D2-KG)")
 	)
 	(segment

Commit message: Added more image
Parts:
- removed R28: 150R, Resistor_SMD:R_0603_1608Metric
- removed Status1: LED, LED_SMD:LED_0805_2012Metric
Connections:
- Blue1 pad 1: Net-(SW3-C) -> Net-(Blue1-Pad1)
- Green1 pad 1: Net-(SW1-C) -> Net-(Green1-Pad1)
- P1 pad A12: Net-(F1-Pad1) -> Net-(Blue1-Pad2)
- P1 pad B12: Net-(F1-Pad1) -> Net-(Blue1-Pad2)
- R1 pad 2: Net-(SW1-B) -> Net-(Green1-Pad1)
- R10 pad 2: Net-(SW1-B) -> Net-(Green1-Pad1)
- R11 pad 2: Net-(SW2-B) -> Net-(R11-Pad2)
- R12 pad 2: Net-(SW3-B) -> Net-(Blue1-Pad1)
- R13 pad 2: Net-(SW1-B) -> Net-(Green1-Pad1)
- R14 pad 2: Net-(SW2-B) -> Net-(R11-Pad2)
- R15 pad 2: Net-(SW3-B) -> Net-(Blue1-Pad1)
- R16 pad 2: Net-(SW1-B) -> Net-(Green1-Pad1)
- R17 pad 2: Net-(SW2-B) -> Net-(R11-Pad2)
- R18 pad 2: Net-(SW3-B) -> Net-(Blue1-Pad1)
- R19 pad 2: Net-(SW1-B) -> Net-(Green1-Pad1)
- R2 pad 2: Net-(SW2-B) -> Net-(R11-Pad2)
- R20 pad 2: Net-(SW2-B) -> Net-(R11-Pad2)
- R21 pad 2: Net-(SW3-B) -> Net-(Blue1-Pad1)
- R22 pad 2: Net-(SW1-B) -> Net-(Green1-Pad1)
- R23 pad 2: Net-(SW2-B) -> Net-(R11-Pad2)
- R24 pad 2: Net-(SW3-B) -> Net-(Blue1-Pad1)
- R25 pad 2: Net-(SW1-B) -> Net-(Green1-Pad1)
- R26 pad 2: Net-(SW2-B) -> Net-(R11-Pad2)
- R27 pad 2: Net-(SW3-B) -> Net-(Blue1-Pad1)
- R3 pad 2: Net-(SW3-B) -> Net-(Blue1-Pad1)
- R4 pad 2: Net-(SW1-B) -> Net-(Green1-Pad1)
- R5 pad 2: Net-(SW2-B) -> Net-(R11-Pad2)
- R6 pad 2: Net-(SW3-B) -> Net-(Blue1-Pad1)
- R7 pad 2: Net-(SW1-B) -> Net-(Green1-Pad1)
- R8 pad 2: Net-(SW2-B) -> Net-(R11-Pad2)
- R9 pad 2: Net-(SW3-B) -> Net-(Blue1-Pad1)
- Red1 pad 1: Net-(SW2-C) -> Net-(R11-Pad2)
Routing:
- net Net-(D1-AB): track 108.0 -> 93.0 mm
- net Net-(Status1-K): track 2.37 -> 0.00 mm
- net Net-(F1-Pad1): vias 3 -> 0
- net Net-(Blue1-Pad2): vias 0 -> 3

Commit message: v1.2 LedCube pcb
Parts:
- removed F1: Polyfuse, Fuse:Fuse_BelFuse_0ZRE0005FF_L8.3mm_W3.8mm
- removed SW1, SW2, SW3: SW_SPDT_321, Button_Switch_THT:SW_DIP_SPSTx01_Slide_6.7x4.1mm_W7.62mm_P2.54mm_LowProfile
- added D10: LED, LED_SMD:LED_0805_2012Metric, B.Cu at (121.0, 85.5)
- added Q1: BC847, Package_TO_SOT_SMD:SOT-23, F.Cu at (96.5, 93.5)
- added Q2: BC847, Package_TO_SOT_SMD:SOT-23, F.Cu at (92.0, 93.5)
- added Q3: BC847, Package_TO_SOT_SMD:SOT-23, F.Cu at (87.5, 93.5)
- added R28: 1000R, Resistor_SMD:R_0603_1608Metric, F.Cu at (95.5, 98.5)
- added R29: 1000R, Resistor_SMD:R_0603_1608Metric, F.Cu at (92.5, 98.5)
- added R30: 1000R, Resistor_SMD:R_0603_1608Metric, F.Cu at (89.5, 98.5)
- added R31: 150R, Resistor_SMD:R_0603_1608Metric, B.Cu at (121.0, 90.0)
- Blue1, Green1, Red1: footprint Potentiometer_THT:Potentiometer_Bourns_3266W_Vertical -> Potentiometer_SMD:Potentiometer_Bourns_3314G_Vertical
- moved Red1 48.3 mm to (87.0, 61.0), turned to 90 degrees
- moved Blue1 41.9 mm to (117.2, 95.8)
- moved Green1 3.10 mm to (114.0, 61.5), turned to 90 degrees
- moved R12 3.05 mm to (97.5, 67.5)
- moved R21 3.01 mm to (108.5, 67.5)
- moved R3 2.64 mm to (85.0, 67.9)
- moved R11 2.55 mm to (97.5, 70.0)
- moved R20 2.51 mm to (108.5, 70.0)
- moved D4 2.43 mm to (103.0, 70.0)
- moved D7 2.38 mm to (114.0, 70.0)
- moved D1 2.14 mm to (91.5, 70.3)
- moved R2 2.14 mm to (85.0, 70.4)
- moved R10 2.05 mm to (97.5, 72.5)
- moved R15 1.65 mm to (97.7, 75.5)
- moved R1 1.58 mm to (85.0, 73.0)
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Connections:
- Blue1 pad 1: Net-(Blue1-Pad1) -> Net-(D1-AB)
- Blue1 pad 3: unconnected-(Blue1-Pad3) -> Net-(D10-K)
- Green1 pad 1: Net-(Green1-Pad1) -> Net-(D1-AB)
- Green1 pad 2: Net-(Blue1-Pad2) -> Net-(Green1-Pad2)
- Green1 pad 3: unconnected-(Green1-Pad3) -> Net-(D10-K)
- P1 pad A12: Net-(Blue1-Pad2) -> Net-(D10-K)
- P1 pad B12: Net-(Blue1-Pad2) -> Net-(D10-K)
- R1 pad 2: Net-(Green1-Pad1) -> Net-(Q1-C)
- R10 pad 2: Net-(Green1-Pad1) -> Net-(Q1-C)
- R11 pad 2: Net-(R11-Pad2) -> Net-(Q2-C)
- R12 pad 2: Net-(Blue1-Pad1) -> Net-(Q3-C)
- R13 pad 2: Net-(Green1-Pad1) -> Net-(Q1-C)
- R14 pad 2: Net-(R11-Pad2) -> Net-(Q2-C)
- R15 pad 2: Net-(Blue1-Pad1) -> Net-(Q3-C)
- R16 pad 2: Net-(Green1-Pad1) -> Net-(Q1-C)
- R17 pad 2: Net-(R11-Pad2) -> Net-(Q2-C)
- R18 pad 2: Net-(Blue1-Pad1) -> Net-(Q3-C)
- R19 pad 2: Net-(Green1-Pad1) -> Net-(Q1-C)
- R2 pad 2: Net-(R11-Pad2) -> Net-(Q2-C)
- R20 pad 2: Net-(R11-Pad2) -> Net-(Q2-C)
- R21 pad 2: Net-(Blue1-Pad1) -> Net-(Q3-C)
- R22 pad 2: Net-(Green1-Pad1) -> Net-(Q1-C)
- R23 pad 2: Net-(R11-Pad2) -> Net-(Q2-C)
- R24 pad 2: Net-(Blue1-Pad1) -> Net-(Q3-C)
- R25 pad 2: Net-(Green1-Pad1) -> Net-(Q1-C)
- R26 pad 2: Net-(R11-Pad2) -> Net-(Q2-C)
- R27 pad 2: Net-(Blue1-Pad1) -> Net-(Q3-C)
- R3 pad 2: Net-(Blue1-Pad1) -> Net-(Q3-C)
- R4 pad 2: Net-(Green1-Pad1) -> Net-(Q1-C)
- R5 pad 2: Net-(R11-Pad2) -> Net-(Q2-C)
- R6 pad 2: Net-(Blue1-Pad1) -> Net-(Q3-C)
- R7 pad 2: Net-(Green1-Pad1) -> Net-(Q1-C)
- R8 pad 2: Net-(R11-Pad2) -> Net-(Q2-C)
- R9 pad 2: Net-(Blue1-Pad1) -> Net-(Q3-C)
- Red1 pad 1: Net-(R11-Pad2) -> Net-(D1-AB)
- Red1 pad 2: Net-(Blue1-Pad2) -> Net-(R29-Pad1)
- Red1 pad 3: unconnected-(Red1-Pad3) -> Net-(D10-K)
Routing:
- net Net-(SW2-B): track 196.1 -> 0.00 mm, vias 9 -> 0
- net Net-(SW3-B): track 189.1 -> 0.00 mm, vias 9 -> 0
- net Net-(D10-K): track 0.00 -> 175.6 mm, vias 0 -> 1
- net Net-(Q2-C): track 0.00 -> 163.5 mm, vias 0 -> 9
- net Net-(Q1-C): track 0.00 -> 137.5 mm, vias 0 -> 9
- net Net-(Q3-C): track 0.00 -> 111.5 mm, vias 0 -> 9
- net Net-(SW1-B): track 104.2 -> 0.00 mm, vias 9 -> 0
- net Net-(R29-Pad1): track 0.00 -> 103.9 mm, vias 0 -> 2
- net Net-(Green1-Pad2): track 0.00 -> 73.5 mm, vias 0 -> 2
- net Net-(Blue1-Pad2): track 95.3 -> 32.5 mm, vias 3 -> 2
- net Net-(D1-AB): track 93.0 -> 147.4 mm
- net Net-(F1-Pad1): track 35.0 -> 0.00 mm
- net Net-(SW2-C): track 14.5 -> 0.00 mm
- net Net-(SW3-C): track 9.98 -> 0.00 mm
- net Net-(SW1-C): track 9.98 -> 0.00 mm
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Other:
- outline, holes or cut-outs redrawn
- board text removed: "+5V"
- board text removed: "-GND"
